File: Logic Probe Ver.1.brd (EAGLE design)
At the start: 160 x 100 mm, 48 parts, among them J5 TST-125-01-G-D, U1 DS90LV047ATM, U2 DS90LV047ATM, U3 DS90LV047ATM, U4 DS90LV047ATM, U5 SN74BCT543DW, U6 SN74BCT543DW

Commit message: PCB Submission
Attempt to fix the comments received for PCB
Routing:
- net N$4: track 10.2 -> 0.00 mm
Other:
- board text added: "+4V"
- board text added: "OUT8-"
- board text added: "OUT9+"
- board text added: "Probe"
Changed lines of the file:
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@@
 <setting verticaltext="up"/>
 </settings>
-<grid distance="12" unitdist="mil" unit="mil" style="lines" multiple="1" display="yes" altdistance="5" altunitdist="mil" altunit="mil"/>
+<grid distance="1" unitdist="mm" unit="mm" style="lines" multiple="1" display="yes" altdistance="5" altunitdist="mil" altunit="mil"/>
 <layers>
 <layer number="1" name="Top" color="4" fill="1" visible="yes" active="yes"/>
@@
 <text x="28.6512" y="24.6888" size="1.778" layer="22" rot="MR0">Jin Feng Lin PCB2.0 </text>
 <text x="28.956" y="21.6408" size="1.778" layer="22" rot="MR0">Logic Analyzer Probe</text>
-<text x="51.2064" y="14.3256" size="1.778" layer="22" rot="MR0">https://github.com/umd-jfl/ECE388Project</text>
+<text x="52.1208" y="14.6304" size="1.778" layer="22" rot="MR0">https://github.com/umd-jfl/ECE388Project</text>
 <text x="29.2608" y="18.5928" size="1.778" layer="22" rot="MR0">11/12/2020</text>
 <text x="67.056" y="64.3128" size="1.778" layer="22" rot="MR180">OUT0+</text>
@@
 <text x="74.676" y="65.532" size="1.778" layer="22" rot="MR0">OUT9-</text>
 <text x="74.676" y="67.9704" size="1.778" layer="22" rot="MR0">OUT8+</text>
+<text x="93" y="70" size="1.778" layer="22" rot="MR0">OUT8-</text>
+<text x="93" y="68" size="1.778" layer="22" rot="MR0">OUT9+</text>
+<text x="74" y="83" size="1.778" layer="22" rot="MR0">Probe</text>
+<text x="74" y="81" size="1.778" layer="22" rot="MR0">GND</text>
+<text x="91" y="83" size="1.778" layer="22" rot="MR0">GND</text>
+<text x="90" y="76" size="1.778" layer="22" rot="MR0">+4V</text>
+<text x="90" y="74" size="1.778" layer="22" rot="MR0">+4V</text>
+<text x="69" y="75" size="1.778" layer="22" rot="MR180">GND</text>
+<text x="69" y="73" size="1.778" layer="22" rot="MR180">GND</text>
+<text x="69" y="59" size="1.778" layer="22" rot="MR180">GND</text>
+<text x="69" y="47" size="1.778" layer="22" rot="MR180">GND</text>
+<text x="69" y="35" size="1.778" layer="22" rot="MR180">GND</text>
+<text x="85" y="24" size="1.778" layer="22" rot="MR180">GND</text>
+<text x="86" y="37" size="1.778" layer="22" rot="MR180">GND</text>
+<text x="86" y="50" size="1.778" layer="22" rot="MR180">GND</text>
+<text x="91" y="60" size="1.778" layer="22" rot="MR0">GND</text>
+<dimension x1="3" y1="15" x2="98" y2="15" x3="50.5" y3="5" textsize="1.778" layer="1"/>
+<dimension x1="92" y1="96" x2="93" y2="9" x3="100.498940625" y3="52.5919375" textsize="1.778" layer="1"/>
 </plain>
 <attributes>
@@
 <wire x1="44.196" y1="45.1104" x2="44.196" y2="45.212" width="0.3048" layer="1"/>
 <via x="44.196" y="45.212" extent="1-16" drill="0.508"/>
-<polygon width="0.3048" layer="1" isolate="0.000509375">
-<vertex x="9.144" y="95.4024"/>
-<vertex x="2.4384" y="88.6968"/>
-<vertex x="2.4384" y="88.392"/>
-<vertex x="2.4384" y="16.1544"/>
-<vertex x="12.192" y="6.4008"/>
-<vertex x="90.8304" y="6.4008"/>
-<vertex x="93.2688" y="8.8392"/>
-<vertex x="99.06" y="14.6304"/>
-<vertex x="99.06" y="15.8496"/>
-<vertex x="99.06" y="88.392"/>
-<vertex x="96.9264" y="90.5256"/>
-<vertex x="92.0496" y="95.4024"/>
+<polygon width="0.1524" layer="1" isolate="0.02">
+<vertex x="3" y="92"/>
+<vertex x="7" y="96"/>
+<vertex x="8" y="96"/>
+<vertex x="92" y="96"/>
+<vertex x="98" y="90"/>
+<vertex x="98" y="14"/>
+<vertex x="93" y="9"/>
+<vertex x="9" y="9"/>
+<vertex x="4" y="14"/>
+<vertex x="3" y="15"/>
 </polygon>
-<polygon width="0.3048" layer="16" isolate="0.000509375">
-<vertex x="10.0584" y="95.7072"/>
-<vertex x="3.048" y="88.6968"/>
-<vertex x="2.1336" y="88.6968"/>
-<vertex x="2.1336" y="16.4592"/>
-<vertex x="12.192" y="6.4008"/>
-<vertex x="90.8304" y="6.4008"/>
-<vertex x="99.06" y="14.6304"/>
-<vertex x="99.06" y="88.392"/>
-<vertex x="92.0496" y="95.4024"/>
+<polygon width="0.1524" layer="16" isolate="0.02">
+<vertex x="3" y="92"/>
+<vertex x="7" y="96"/>
+<vertex x="92" y="96"/>
+<vertex x="98" y="90"/>
+<vertex x="98" y="14"/>
+<vertex x="93" y="9"/>
+<vertex x="9" y="9"/>
+<vertex x="3" y="15"/>
 </polygon>
 </signal>
@@
 <wire x1="33.655" y1="45.085" x2="34.29" y2="44.45" width="0.3048" layer="1"/>
 <wire x1="34.29" y1="44.45" x2="37.15" y2="44.45" width="0.3048" layer="1"/>
-</signal>
-<signal name="N$4">
-<contactref element="R9" pad="2"/>
-<contactref element="U6" pad="22"/>
-<wire x1="29.845" y1="46.355" x2="27.5" y2="46.355" width="0.3048" layer="1"/>
-<wire x1="35.88" y1="50.8" x2="34.29" y2="50.8" width="0.3048" layer="1"/>
-<wire x1="34.29" y1="50.8" x2="29.845" y2="46.355" width="0.3048" layer="1"/>
 </signal>
 <signal name="N$9">
@@
 <wire x1="16.7386" y1="37.465" x2="16.1544" y2="36.8808" width="0.3048" layer="1"/>
 </signal>
+<signal name="N$4">
+<contactref element="R9" pad="2"/>
+<contactref element="U6" pad="22"/>
+<wire x1="27.5" y1="46.355" x2="35.88" y2="50.8" width="0" layer="19" extent="1-1"/>
+</signal>
 </signals>
